File: pcb-te/power.kicad_sch (KiCad schematic)
At the start: 24 parts, among them U1 NCP163AFCT250T2G, U2 ADP220ACBZ-1812R7, U3 ADP220ACBZ-1812R7

Commit message: Added new fields (OEPS PN, MPN, and Type) to all components.
Parts:
- C1, C10, C11, C2, C4, C5, C8, C9: MPN (none) -> CL03A105MO3NRNH; OEPS PN (none) -> OEPS010036; Type (none) -> SMD
- C? (x2): MPN (none) -> CL05A106MP5NUNC; OEPS PN (none) -> OEPS010038; Type (none) -> SMD
- C?: MPN (none) -> GRM033R61E104KE14J; OEPS PN (none) -> OEPS010035; Type (none) -> SMD
- L1: MPN (none) -> CBC3225T101MR; OEPS PN (none) -> OEPS040010; Type (none) -> SMD
- L2: MPN (none) -> ASMPH-0805-4R7M-T; OEPS PN (none) -> OEPS040007; Type (none) -> SMD
- R3, R4: MPN (none) -> RC0201FR-072KL; OEPS PN (none) -> OEPS020067; Type (none) -> SMD
- R5: MPN (none) -> CRCW02017K15FKED; OEPS PN (none) -> OEPS020058; Type (none) -> SMD
- U1: MPN (none) -> NCP163AFCT250T2G; OEPS PN (none) -> OEPS080062; Type (none) -> SMD
- U2, U3: MPN (none) -> ADP220ACBZ-1812R7; OEPS PN (none) -> OEPS080061; Type (none) -> SMD
- U?: MPN (none) -> TPS3839E16DQNT; OEPS PN (none) -> OEPS080060; Type (none) -> SMD
