File: pcb-te/perpherials.kicad_sch (KiCad schematic)
At the start: 9 parts, among them J5 5050700622, U8 M24C64-FCS6TP/K, U9 BNO055

Commit message: Added new fields (OEPS PN, MPN, and Type) to all components.
Parts:
- C32, C33, C34, C35: MPN (none) -> GRM033R61E104KE14J; OEPS PN (none) -> OEPS010035; Type (none) -> SMD
- J5: MPN (none) -> 5050700622; OEPS PN (none) -> OEPS070049; Type (none) -> SMD
- J?: Type (none) -> SMD
- J?: Type (none) -> TH
- U8: MPN (none) -> M24C64-FCS6TP/K; OEPS PN (none) -> OEPS080050; Type (none) -> SMD
- U9: MPN (none) -> BNO055; OEPS PN (none) -> OEPS080063; Type (none) -> SMD
Changed lines of the file:
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@@
+      (effects (font (size 1.27 1.27)) hide)
+    )
+    (property "MPN" "BNO055" (at 129.54 127 0)
+      (effects (font (size 1.27 1.27)) hide)
+    )
+    (property "OEPS PN" "OEPS080063" (at 129.54 127 0)
+      (effects (font (size 1.27 1.27)) hide)
+    )
+    (property "Type" "SMD" (at 129.54 127 0)
+      (effects (font (size 1.27 1.27)) hide)
+    )
+    (property "test" "" (at 129.54 127 0)
       (effects (font (size 1.27 1.27)) hide)
     )
@@
       (effects (font (size 1.27 1.27)) hide)
     )
+    (property "MPN" "5050700622" (at 214.63 125.73 0)
+      (effects (font (size 1.27 1.27)) hide)
+    )
+    (property "OEPS PN" "OEPS070049" (at 214.63 125.73 0)
+      (effects (font (size 1.27 1.27)) hide)
+    )
+    (property "Type" "SMD" (at 214.63 125.73 0)
+      (effects (font (size 1.27 1.27)) hide)
+    )
+    (property "test" "" (at 214.63 125.73 0)
+      (effects (font (size 1.27 1.27)) hide)
+    )
     (pin "1")
     (pin "2")
@@
       (effects (font (size 1.27 1.27)) hide)
     )
+    (property "MPN" "GRM033R61E104KE14J" (at 217.17 59.69 0)
+      (effects (font (size 1.27 1.27)) hide)
+    )
+    (property "OEPS PN" "OEPS010035" (at 217.17 59.69 0)
+      (effects (font (size 1.27 1.27)) hide)
+    )
+    (property "Type" "SMD" (at 217.17 59.69 0)
+      (effects (font (size 1.27 1.27)) hide)
+    )
+    (property "test" "" (at 217.17 59.69 0)
+      (effects (font (size 1.27 1.27)) hide)
+    )
     (pin "1")
     (pin "2")
@@
     )
     (property "Tolerance" "" (at 198.12 59.69 0)
+      (effects (font (size 1.27 1.27)) hide)
+    )
+    (property "MPN" "M24C64-FCS6TP/K" (at 198.12 59.69 0)
+      (effects (font (size 1.27 1.27)) hide)
+    )
+    (property "OEPS PN" "OEPS080050" (at 198.12 59.69 0)
+      (effects (font (size 1.27 1.27)) hide)
+    )
+    (property "Type" "SMD" (at 198.12 59.69 0)
+      (effects (font (size 1.27 1.27)) hide)
+    )
+    (property "test" "" (at 198.12 59.69 0)
       (effects (font (size 1.27 1.27)) hide)
     )
@@
       (effects (font (size 1.27 1.27)) hide)
     )
+    (property "MPN" "GRM033R61E104KE14J" (at 87.63 110.49 0)
+      (effects (font (size 1.27 1.27)) hide)
+    )
+    (property "OEPS PN" "OEPS010035" (at 87.63 110.49 0)
+      (effects (font (size 1.27 1.27)) hide)
+    )
+    (property "Type" "SMD" (at 87.63 110.49 0)
+      (effects (font (size 1.27 1.27)) hide)
+    )
+    (property "test" "" (at 87.63 110.49 0)
+      (effects (font (size 1.27 1.27)) hide)
+    )
     (pin "1")
     (pin "2")
@@
     )
     (property "Tolerance" "" (at 146.05 59.69 0)
+      (effects (font (size 1.27 1.27)) hide)
+    )
+    (property "MPN" "" (at 146.05 59.69 0)
+      (effects (font (size 1.27 1.27)) hide)
+    )
+    (property "OEPS PN" "" (at 146.05 59.69 0)
+      (effects (font (size 1.27 1.27)) hide)
+    )
+    (property "Type" "SMD" (at 146.05 59.69 0)
+      (effects (font (size 1.27 1.27)) hide)
+    )
+    (property "test" "" (at 146.05 59.69 0)
       (effects (font (size 1.27 1.27)) hide)
     )
@@
       (effects (font (size 1.27 1.27)) hide)
     )
+    (property "MPN" "GRM033R61E104KE14J" (at 160.02 110.49 0)
+      (effects (font (size 1.27 1.27)) hide)
+    )
+    (property "OEPS PN" "OEPS010035" (at 160.02 110.49 0)
+      (effects (font (size 1.27 1.27)) hide)
+    )
+    (property "Type" "SMD" (at 160.02 110.49 0)
+      (effects (font (size 1.27 1.27)) hide)
+    )
+    (property "test" "" (at 160.02 110.49 0)
+      (effects (font (size 1.27 1.27)) hide)
+    )
     (pin "1")
     (pin "2")
@@
       (effects (font (size 1.27 1.27)) hide)
     )
+    (property "MPN" "GRM033R61E104KE14J" (at 149.86 144.78 0)
+      (effects (font (size 1.27 1.27)) hide)
+    )
+    (property "OEPS PN" "OEPS010035" (at 149.86 144.78 0)
+      (effects (font (size 1.27 1.27)) hide)
+    )
+    (property "Type" "SMD" (at 149.86 144.78 0)
+      (effects (font (size 1.27 1.27)) hide)
+    )
+    (property "test" "" (at 149.86 144.78 0)
+      (effects (font (size 1.27 1.27)) hide)
+    )
     (pin "1")
     (pin "2")
@@
       (effects (font (size 1.27 1.27)) hide)
     )
+    (property "MPN" "" (at 96.52 58.42 0)
+      (effects (font (size 1.27 1.27)) hide)
+    )
+    (property "OEPS PN" "" (at 96.52 58.42 0)
+      (effects (font (size 1.27 1.27)) hide)
+    )
+    (property "Type" "TH" (at 96.52 58.42 0)
+      (effects (font (size 1.27 1.27)) hide)
+    )
+    (property "test" "" (at 96.52 58.42 0)
+      (effects (font (size 1.27 1.27)) hide)
+    )
