File: pcb-te/serializer.kicad_sch (KiCad schematic)
At the start: 25 parts, among them U5 DS90UB933TRTVTQ1

Commit message: Added new fields (OEPS PN, MPN, and Type) to all components.
Parts:
- C12, C14, C16, C19, C22: MPN (none) -> GRM033R71E103KE14D; OEPS PN (none) -> OEPS010037; Type (none) -> SMD
- C13, C15, C17, C20, C23, C25: MPN (none) -> GRM033R61E104KE14J; OEPS PN (none) -> OEPS010035; Type (none) -> SMD
- C18, C21, C24: MPN (none) -> CL05A106MP5NUNC; OEPS PN (none) -> OEPS010038; Type (none) -> SMD
- C26: MPN (none) -> CC0201KRX5R8BB473; OEPS PN (none) -> OEPS010031; Type (none) -> SMD
- C27: MPN (none) -> CL03A105MO3NRNH; OEPS PN (none) -> OEPS010036; Type (none) -> SMD
- D1: MPN (none) -> SML-P11UTT86R; OEPS PN (none) -> OEPS030014; Type (none) -> SMD
- L3, L4: MPN (none) -> BLF03RD501GZED; OEPS PN (none) -> OEPS040006; Type (none) -> SMD
- R10: MPN (none) -> RC0201FR-0749R9L; OEPS PN (none) -> OEPS020068; Type (none) -> SMD
- R6: MPN (none) -> RC0201FR-071KL; OEPS PN (none) -> OEPS020065; Type (none) -> SMD
- R7, R8, R9: MPN (none) -> CRCW020110K0FNED; OEPS PN (none) -> OEPS020066; Type (none) -> SMD
- U5: MPN (none) -> DS90UB933TRTVTQ1; OEPS PN (none) -> OEPS080064; Type (none) -> SMD
